Commit message: Updated URDF

File: ros2_cobot/src/urdf/Cobot.urdf (robot description, URDF)
Before this commit: robot Cobot, 5 links, 4 joints
Links:
- removed link Wrist
- added link Link4, mass 0.0101757375861059; collision mesh filename=package://urdf/meshes/Link4.STL; visual mesh filename=package://urdf/meshes/Link4.STL
- link Link1: geometry collision mesh filename=package://urdf/meshes/Link1.STL; visual mesh filename=package://urdf/meshes/Link1.STL
- link Link2: mass 0.12624 -> 0.126238291044564; geometry collision mesh filename=package://urdf/meshes/Link2.STL; visual mesh filename=package://urdf/meshes/Link2.STL
- link Link3: mass 0.11268 -> 0.11268362796461; geometry collision mesh filename=package://urdf/meshes/Link3.STL; visual mesh filename=package://urdf/meshes/Link3.STL
- link base_link: mass 0.26278 -> 0.262781517647469; geometry collision mesh filename=package://urdf/meshes/base_link.STL; visual mesh filename=package://urdf/meshes/base_link.STL
Joints:
- removed joint WristJoint
- added joint Joint3: type revolute, parent Link3, child Link4, origin xyz=0 -0.00020911 0.1673 rpy=0 0 0, axis 1 0 0, limit lower=0 upper=0 effort=0 velocity=0
- joint Joint0: axis 0 0 1 -> 0 0 0; limit lower=0 upper=6.2383 effort=1.47 velocity=4.7123 -> lower=0 upper=0 effort=0 velocity=0; origin xyz=0 0 0.064 rpy=0 0 -0.047986 -> xyz=-0.012386 0.0016827 0.0463 rpy=0 0 -0.13503
- joint Joint1: limit lower=-1.4835 upper=2.8798 effort=1.47 velocity=4.7123 -> lower=0 upper=0 effort=0 velocity=0; origin xyz=0 0.00062634 0.0712 rpy=-0.67663 0 0 -> xyz=0 0.00062634 0.0889 rpy=0 0 0
- joint Joint2: limit lower=-4.0143 upper=0.2618 effort=1.47 velocity=4.7123 -> lower=0 upper=0 effort=0 velocity=0; origin xyz=0 -0.00020923 0.2073 rpy=1.9015 0 0 -> xyz=0 -0.00020923 0.2073 rpy=0 0 0

Commit message: Update: Trying to make robot dance

File: ros2_cobot/src/urdf/Cobot.urdf (robot description, URDF)
Before this commit: robot Cobot, 5 links, 4 joints
Joints:
- joint Joint0: limit lower=0 upper=0 effort=0 velocity=0 -> lower=0 upper=0 effort=1.47 velocity=4.7123
- joint Joint1: limit lower=0 upper=0 effort=0 velocity=0 -> lower=0 upper=0 effort=1.47 velocity=4.7123
- joint Joint2: limit lower=0 upper=0 effort=0 velocity=0 -> lower=0 upper=0 effort=1.47 velocity=4.7123
- joint Joint3: limit lower=0 upper=0 effort=0 velocity=0 -> lower=0 upper=0 effort=1.47 velocity=4.7123
