Commit message: Update: Cobot control added: joints set/read, rough pose set/read, started trajectory planner

File: ros2_cobot/src/cobot_description/urdf/Cobot.urdf (robot description, URDF)
Before this commit: robot Cobot, 5 links, 4 joints
Joints:
- joint Joint0: axis 0 0 0 -> 0 0 1; limit lower=0 upper=0 effort=1.47 velocity=4.7123 -> lower=-3.14159 upper=3.14159 effort=1.47 velocity=4.7123; origin xyz=-0.012386 0.0016827 0.0463 rpy=0 0 -0.13503 -> xyz=0.0 0.0 0.0463 rpy=0 0 -0.13503
- joint Joint1: limit lower=0 upper=0 effort=1.47 velocity=4.7123 -> lower=-1.48353 upper=1.48353 effort=1.47 velocity=4.7123
- joint Joint2: limit lower=0 upper=0 effort=1.47 velocity=4.7123 -> lower=-2.09440 upper=2.09440 effort=1.47 velocity=4.7123
- joint Joint3: limit lower=0 upper=0 effort=1.47 velocity=4.7123 -> lower=-1.91986 upper=1.91986 effort=1.47 velocity=4.7123
